File: Follower.kicad_pcb (KiCad board)
At the start: 2 copper layers, 40 x 80 mm, 39 parts, among them J1 AVR-ISP-6, J2 Serial-328P, J3 Conn_01x05_Pin, J4 Conn_02x08_Odd_Even, J6 Conn_01x04_Pin, J8 HallSensor, J9 Conn_01x04_Pin, SW1 AVR RESET, U1 ATmega328P-A, U2 TPS54331DDAR, U3 ULN2003A, Y1 16MHz

Commit message: 1.0.0
Parts:
- R3: value 51.1 -> 120
- SW1: value AVR RESET -> RESET
Routing:
- net /D3: track 18.8 -> 49.1 mm, vias 1 -> 0
- net GND: track 0.00 -> 26.8 mm, vias 0 -> 4
- net /A1: track 31.1 -> 17.2 mm, vias 1 -> 0
- net /A2: track 27.7 -> 17.4 mm, vias 1 -> 0
- net /D2: track 33.2 -> 23.2 mm
- net /D9: track 0.00 -> 9.38 mm, vias 0 -> 2
- net +3V3: track 131.4 -> 123.4 mm, vias 0 -> 1
- net /D7: track 34.3 -> 37.5 mm
- net /RESET: track 72.3 -> 74.9 mm
- net /A0: track 19.5 -> 17.2 mm, vias 1 -> 0
- net /D4: track 18.4 -> 16.8 mm
- net /D0: track 18.0 -> 19.2 mm, vias 0 -> 1
- net /A4/SDA: track 85.0 -> 85.1 mm, vias 0 -> 1
Other:
- board text added: "AfterAI Flaps Follower 1.0.0"
- board text removed: "AfterAI Flaps Follower 1.0.dev"
