File: Follower.kicad_sch (KiCad schematic)
At the start: 39 parts, among them J1 AVR-ISP-6, J2 Serial-328P, J3 Conn_01x05_Pin, J4 Conn_02x08_Odd_Even, J6 Conn_01x04_Pin, J8 HallSensor, J9 Conn_01x04_Pin, SW1 RESET, U1 ATmega328P-A, U2 TPS54331DDAR, U3 ULN2003A, Y1 16MHz

Commit message: 1.0.0
Parts:
- J4: LCSC (none) -> C5383108; lcsc C68234 -> (none)
- R3: value 51.1 -> 120; LCSC C3015638 -> C25079
- U2: LCSC (none) -> C90761
